Commit message: [UPDATE] Added TCP & Payload load

File: ur_description/urdf/inc/ur_macro.xacro (robot description, xacro)
@@ -52,4 +52,7 @@
     pitch_EE:=0
     yaw_EE:=0
+    roll_Last_Link:=0
+    pitch_Last_Link:=0
+    yaw_Last_Link:=0
     joint_limits_parameters_file
     kinematics_parameters_file
@@ -316,6 +319,5 @@
     <link name="${prefix}rpwc_last_robot_link"/>
     <joint name="${prefix}flange-rpwc_last_robot_link" type="fixed">
-      <!-- default toolframe: X+ left, Y+ up, Z+ front -->
-      <origin xyz="0 0 0" rpy="0 ${pi/2.0} 0"/>
+      <origin xyz="0 0 0" rpy="${roll_Last_Link} ${pitch_Last_Link} ${yaw_Last_Link}"/>
       <parent link="${prefix}flange"/>
       <child link="${prefix}rpwc_last_robot_link"/>

File: ur_description/urdf/ur.xacro (robot description, xacro)
@@ -15,4 +15,7 @@
    <xacro:arg name="pitch_EE" default="0"/>
    <xacro:arg name="yaw_EE" default="0"/>
+   <xacro:arg name="roll_Last_Link" default="0"/>
+   <xacro:arg name="pitch_Last_Link" default="0"/>
+   <xacro:arg name="yaw_Last_Link" default="0"/>
    <!-- legal values:
          - hardware_interface/PositionJointInterface
@@ -33,4 +36,7 @@
      pitch_EE="$(arg pitch_EE)"
      yaw_EE="$(arg yaw_EE)"
+     roll_Last_Link="$(arg roll_Last_Link)"
+     pitch_Last_Link="$(arg pitch_Last_Link)"
+     yaw_Last_Link="$(arg yaw_Last_Link)"
      joint_limits_parameters_file="$(arg joint_limit_params)"
      kinematics_parameters_file="$(arg kinematics_params)"

Commit message: [FIX] Fixed tool rotation

File: ur_description/urdf/inc/ur_macro.xacro (robot description, xacro)
@@ -317,17 +317,4 @@
       <origin xyz="0 0 0" rpy="0 ${-pi/2.0} ${-pi/2.0}" />
     </joint>
-    <link name="${prefix}rpwc_last_robot_link"/>
-    <joint name="${prefix}flange-rpwc_last_robot_link" type="fixed">
-      <origin xyz="0 0 0" rpy="${roll_Last_Link} ${pitch_Last_Link} ${yaw_Last_Link}"/>
-      <parent link="${prefix}flange"/>
-      <child link="${prefix}rpwc_last_robot_link"/>
-    </joint>
-    <link name="${prefix}rpwc_EE"/>
-    <joint name="${prefix}rpwc_last_robot_link-rpwc_EE" type="fixed">
-      <origin xyz="${x_pos_EE} ${y_pos_EE} ${z_pos_EE}" rpy="${roll_EE} ${pitch_EE} ${yaw_EE}" />
-      <!-- <origin xyz="$(arg x_pos_EE) $(arg y_pos_EE) $(arg z_pos_EE)" rpy="$(arg roll_EE) $(arg pitch_EE) $(arg yaw_EE)" /> -->
-      <parent link="${prefix}rpwc_last_robot_link"/>
-      <child link="${prefix}rpwc_EE"/>
-    </joint>
     <!-- ROS-Industrial 'tool0' frame: all-zeros tool frame -->
     <link name="${prefix}tool0"/>
@@ -338,4 +325,17 @@
       <child link="${prefix}tool0"/>
     </joint>
+    <link name="${prefix}rpwc_last_robot_link"/>
+    <joint name="${prefix}tool0-rpwc_last_robot_link" type="fixed">
+      <origin xyz="0 0 0" rpy="${roll_Last_Link} ${pitch_Last_Link} ${yaw_Last_Link}"/>
+      <parent link="${prefix}tool0"/>
+      <child link="${prefix}rpwc_last_robot_link"/>
+    </joint>
+    <link name="${prefix}rpwc_EE"/>
+    <joint name="${prefix}rpwc_last_robot_link-rpwc_EE" type="fixed">
+      <origin xyz="${x_pos_EE} ${y_pos_EE} ${z_pos_EE}" rpy="${roll_EE} ${pitch_EE} ${yaw_EE}" />
+      <!-- <origin xyz="$(arg x_pos_EE) $(arg y_pos_EE) $(arg z_pos_EE)" rpy="$(arg roll_EE) $(arg pitch_EE) $(arg yaw_EE)" /> -->
+      <parent link="${prefix}rpwc_last_robot_link"/>
+      <child link="${prefix}rpwc_EE"/>
+    </joint>
   </xacro:macro>
 </robot>

Commit message: [FIXED] swapped base and base_link frame; rebuilded moveit config;

File: ur_description/urdf/inc/ur_macro.xacro (robot description, xacro)
@@ -73,4 +73,5 @@
     <xacro:ur_arm_transmission prefix="${prefix}" hw_interface="${transmission_hw_interface}" />
     <!-- links: main serial chain -->
+    <link name="${prefix}base"/>
     <link name="${prefix}base_link"/>
     <link name="${prefix}base_link_inertia">
@@ -216,4 +217,14 @@
     </link>
     <!-- joints: main serial chain -->
+    <joint name="${prefix}base-base_link" type="fixed">
+      <!-- Note the rotation over Z of pi radians: as base_link is REP-103
+           aligned (ie: has X+ forward, Y+ left and Z+ up), this is needed
+           to correctly align 'base' with the 'Base' coordinate system of
+           the UR controller.
+      -->
+      <origin xyz="0 0 0" rpy="0 0 ${pi}"/>
+      <parent link="${prefix}base"/>
+      <child link="${prefix}base_link"/>
+    </joint>
     <joint name="${prefix}base_link-base_link_inertia" type="fixed">
       <parent link="${prefix}base_link" />
@@ -298,16 +309,4 @@
       <dynamics damping="0" friction="0"/>
     </joint>
-    <!-- ROS-Industrial 'base' frame: base_link to UR 'Base' Coordinates transform -->
-    <link name="${prefix}base"/>
-    <joint name="${prefix}base_link-base_fixed_joint" type="fixed">
-      <!-- Note the rotation over Z of pi radians: as base_link is REP-103
-           aligned (ie: has X+ forward, Y+ left and Z+ up), this is needed
-           to correctly align 'base' with the 'Base' coordinate system of
-           the UR controller.
-      -->
-      <origin xyz="0 0 0" rpy="0 0 ${pi}"/>
-      <parent link="${prefix}base_link"/>
-      <child link="${prefix}base"/>
-    </joint>
     <!-- ROS-Industrial 'flange' frame: attachment point for EEF models -->
     <link name="${prefix}flange" />

File: ur_description/urdf/ur10e.urdf (robot description, URDF)
Before this commit: robot ur10e_robot, 13 links, 12 joints
Joints:
- removed joint base_link-base_fixed_joint
- added joint base-base_link: type fixed, parent base, child base_link, origin xyz=0 0 0 rpy=0 0 3.141592653589793

File: ur_moveit_config/ur10e_moveit_config/config/ur10e_robot.srdf.xacro (robot description, xacro)
@@ -4,5 +4,5 @@
     <!-- GROUPS -->
     <group name="ur10e_arm">
-        <chain base_link="$(arg prefix)base_link" tip_link="$(arg prefix)rpwc_EE"/>
+        <chain base_link="$(arg prefix)base" tip_link="$(arg prefix)rpwc_EE"/>
     </group>
     <!-- GROUP STATES -->
@@ -16,5 +16,5 @@
     </group_state>
     <!-- VIRTUAL JOINT -->
-    <virtual_joint name="$(arg prefix)virtual_joint" type="fixed" parent_frame="$(arg prefix)world" child_link="$(arg prefix)base_link"/>
+    <virtual_joint name="$(arg prefix)virtual_joint" type="fixed" parent_frame="$(arg prefix)world" child_link="$(arg prefix)base"/>
     <!-- DISABLE COLLISIONS -->
     <disable_collisions link1="$(arg prefix)base_link_inertia" link2="$(arg prefix)shoulder_link" reason="Adjacent"/>
